File: Langstone-Soundcard.kicad_pcb (KiCad board)
At the start: 2 copper layers, 66.7 x 66.7 mm, 27 parts, among them J1 NF_IN, J2 USB, J3 NF_OUT, SW1 HID, U1 PCM2902, Y1 12MHz

Commit message: Designregeln OK
Parts:
- moved C3 30.8 mm to (116.8, 89.9), turned to 180 degrees
- moved R8 30.4 mm to (147.8, 94.7), turned to 0 degrees
- moved C8 23.8 mm to (125.7, 104.0), turned to 180 degrees
- moved C7 23.0 mm to (125.7, 107.8), turned to 180 degrees
- moved C4 11.3 mm to (134.9, 84.8), turned to -90 degrees
- moved C12 8.65 mm to (139.7, 90.7)
- moved C9 5.27 mm to (140.0, 84.8), turned to 90 degrees
- moved C10 2.38 mm to (139.4, 101.3)
- moved R4 2.17 mm to (116.8, 92.7)
- moved C5 1.77 mm to (116.8, 96.0)
- moved C11 1.06 mm to (139.4, 103.9)
- moved R7 0.26 mm to (116.9, 87.0)
- turned Y1 to -90 degrees
Routing:
- net Net-(C13-Pad1): track 0.00 -> 50.2 mm
- net Net-(R1-Pad1): track 0.00 -> 36.5 mm, vias 0 -> 2
- net GND: track 0.00 -> 33.9 mm, vias 0 -> 11
- net Net-(J2-Pad2): track 0.00 -> 29.0 mm
- net Net-(C4-Pad2): track 0.00 -> 28.9 mm, vias 0 -> 2
- net Net-(C12-Pad1): track 0.00 -> 28.3 mm
- net Net-(J2-Pad3): track 0.00 -> 24.0 mm
- net Net-(SW1-Pad6): track 0.00 -> 22.5 mm
- net Net-(J2-Pad4): track 0.00 -> 22.5 mm
- net Net-(SW1-Pad5): track 0.00 -> 21.3 mm
- net Net-(SW1-Pad4): track 0.00 -> 19.7 mm
- net Net-(C7-Pad1): track 0.00 -> 13.8 mm
- net Net-(C6-Pad1): track 0.00 -> 13.0 mm
- net Net-(R6-Pad2): track 0.00 -> 12.4 mm
- net Net-(C8-Pad1): track 0.00 -> 11.3 mm
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- added copper zone on B.Cu, net GND
